Commit message: code update

File: Final_catkin/src/lab2andDriver/drivers/universal_robot/ur_description/urdf/block_spawn.urdf (robot description, URDF)
Before this commit: robot block, 1 links, 0 joints
Links:
- link base_link: mass 0.2 -> 0.4

File: Final_catkin/src/lab2andDriver/drivers/universal_robot/ur_description/urdf/block_spawn2.urdf (robot description, URDF)
Before this commit: robot block, 1 links, 0 joints
Links:
- link base_link: mass 0.2 -> 0.4
